File: Membase/EAGLE/PCE128_Rev_C2_Main/PCE128_rev_C2.brd (EAGLE design)
At the start: 36.2 x 56.5 mm, 32 parts, among them IC1 SN74LVC2T45DCTR, IC2 SN74LVC2T45DCTR, IC3 SN74LVC2T45DCTR, IC5 SN74HC157D, J2 MD-80SGK, J3 MD-80SGK

Commit message: Updated to rev. C boards (and PC Board case)
Parts:
- IC1, IC2, IC3: value SN74LVC2T45DCTR -> SN74LVC2T45DCUR; device SamacSys_Parts:SOP65P400X130-8N -> PC-Engine:SOP50P310X90-8N
- moved R3 15.8 mm to (6.10, 27.2)
- moved R2 15.7 mm to (4.95, 27.2)
- moved R15 12.4 mm to (16.1, 18.8), turned to 0 degrees
- moved R1 11.1 mm to (19.4, 18.8), turned to 0 degrees
- moved C10 0.89 mm to (9.91, 23.9)
- moved C3 0.89 mm to (28.8, 22.2)
- moved C9 0.89 mm to (13.1, 23.9)
- moved J4 0.89 mm to (10.7, 36.3)
- moved C1 0.89 mm to (12.7, 29.3)
- moved C2 0.89 mm to (9.65, 29.3)
- moved C6 0.89 mm to (29.2, 29.6)
- moved C7 0.89 mm to (25.9, 29.6)
- moved IC1 0.89 mm to (11.3, 26.4)
- moved IC2 0.89 mm to (27.6, 32.0)
- moved IC3 0.89 mm to (11.3, 31.9)
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Routing:
- net N$5: track 8.66 -> 27.6 mm
- net N$4: track 8.69 -> 26.8 mm
- net N$2: track 31.1 -> 13.8 mm
- net D11: track 29.5 -> 13.8 mm
- net N$36: track 8.63 -> 22.6 mm
- net N$1: track 8.69 -> 21.0 mm
- net D6: track 14.1 -> 2.41 mm
- net D10: track 13.0 -> 2.47 mm
- net GND: track 200.0 -> 202.9 mm
- net +5V: track 112.8 -> 114.8 mm
- net D2_IN: track 34.8 -> 36.3 mm
- net CLR: track 60.9 -> 62.2 mm
- net D3_IN: track 38.8 -> 40.1 mm
- net +3V3: track 43.9 -> 45.0 mm
- net D1_IN: track 38.7 -> 39.3 mm
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Other:
- board size 36.2 x 56.5 mm -> 36.2 x 57.4 mm
- board text added: "PCE128, rev. C2"
- board text removed: "PCE128, rev. B"
