File: Membase/EAGLE/PCE128_Rev_C2_Main/PCE128_rev_C2.sch (EAGLE design)
At the start: 32 parts, among them IC1 SN74LVC2T45DCTR, IC2 SN74LVC2T45DCTR, IC3 SN74LVC2T45DCTR, IC5 SN74HC157D, J2 MD-80SGK, J3 MD-80SGK

Commit message: Updated to rev. C boards (and PC Board case)
Parts:
- IC1, IC2, IC3: value SN74LVC2T45DCTR -> SN74LVC2T45DCUR; device SamacSys_Parts:SN74LVC2T45DCTR -> PC-Engine:SN74LVC2T45DCUR
Changed lines of the file:
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@@
 <part name="FRAME1" library="frames" library_urn="urn:adsk.eagle:library:229" deviceset="FRAME_A_L" device="" value="Mini-DIN 8 breakout"/>
 <part name="J2" library="SamacSys_Parts" deviceset="MD-80SGK" device=""/>
-<part name="IC2" library="SamacSys_Parts" deviceset="SN74LVC2T45DCTR" device=""/>
+<part name="IC2" library="PC-Engine" deviceset="SN74LVC2T45DCUR" device=""/>
 <part name="GND1" library="supply1" deviceset="GND" device=""/>
 <part name="GND2" library="supply1" deviceset="GND" device=""/>
@@
 <part name="R3" library="resistor" library_urn="urn:adsk.eagle:library:348" deviceset="R-US_" device="R0402" package3d_urn="urn:adsk.eagle:package:26058/2" value="3.3K"/>
 <part name="J3" library="SamacSys_Parts" deviceset="MD-80SGK" device=""/>
-<part name="IC1" library="SamacSys_Parts" deviceset="SN74LVC2T45DCTR" device=""/>
+<part name="IC1" library="PC-Engine" deviceset="SN74LVC2T45DCUR" device=""/>
 <part name="GND13" library="supply1" deviceset="GND" device=""/>
 <part name="GND14" library="supply1" deviceset="GND" device=""/>
@@
 <part name="R23" library="resistor" library_urn="urn:adsk.eagle:library:348" deviceset="R-US_" device="R0402" package3d_urn="urn:adsk.eagle:package:26058/2" value="47K"/>
 <part name="R24" library="resistor" library_urn="urn:adsk.eagle:library:348" deviceset="R-US_" device="R0402" package3d_urn="urn:adsk.eagle:package:26058/2" value="47K"/>
-<part name="IC3" library="SamacSys_Parts" deviceset="SN74LVC2T45DCTR" device=""/>
+<part name="IC3" library="PC-Engine" deviceset="SN74LVC2T45DCUR" device=""/>
 <part name="C1" library="resistor" library_urn="urn:adsk.eagle:library:348" deviceset="C-US" device="C0402" package3d_urn="urn:adsk.eagle:package:23626/2" value="0.1uF"/>
 <part name="C2" library="resistor" library_urn="urn:adsk.eagle:library:348" deviceset="C-US" device="C0402" package3d_urn="urn:adsk.eagle:package:23626/2" value="0.1uF"/>
